Commit message: still not working. Functional up to including new xacro links.

File: urdf/lab4_xacro.xacro (robot description, xacro)
@@ -2,8 +2,14 @@
 <robot xmlns:xacro="http://www.ros.org/wiki/xacro" name="navvis">
 	<xacro:include filename="$(find navvis_description)/urdf/robot_description.xacro" />
+	<link name="base_link" />
 	<joint name="base_link_to_base_joint" type="fixed">
 		<parent link="base_link" />
 		<child link="base" />
 		<origin xyz="0.0 0.0 0.0" rpy="3.1405788 0.0034281 3.1382064" />
+	</joint>
+	<joint name="base_link_to_imu_joint" type="fixed">
+		<parent link="base_link" />
+		<child link="imu" />
+		<origin xyz="0 0 0" rpy="3.1405788 0.0034281 3.1382064" />
 	</joint>
 	<link name="imu">
@@ -15,5 +21,5 @@
 		<collision>
 		<geometry>
-		<sphere radius="0.1">
+		<sphere radius="0.1" />
 		</geometry>
 		</collision>

Commit message: revised code. still not functional

File: urdf/lab4_xacro.xacro (robot description, xacro)
@@ -6,5 +6,5 @@
 		<parent link="base_link" />
 		<child link="base" />
-		<origin xyz="0.0 0.0 0.0" rpy="3.1405788 0.0034281 3.1382064" />
+		<origin xyz="0.07 0.0 1.792" rpy="0.0 ${pi} 0.0" />
 	</joint>
 	<joint name="base_link_to_imu_joint" type="fixed">
